File: OpenTama.sch (KiCad schematic (older format))
At the start: 62 parts, among them J1 Conn_01x09, J2 Conn_01x14, J3 Conn_01x07, J4 USB_C_Receptacle_USB2.0, J5 Conn_01x14, Q1 BSS138, Q2 BSS138, Q3 BSS84, SW1 LEFT, SW2 MIDDLE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

Commit message: Use LCSC instead of JLCPCB in symbol props
Parts:
- C1: JLCPCB C29823 -> (none); LCSC (none) -> C29823
- C10, C5, C8, C9: JLCPCB C1525 -> (none); LCSC (none) -> C1525
- C11: JLCPCB C1615 -> (none); LCSC (none) -> C1615
- C12: JLCPCB C15849 -> (none); LCSC (none) -> C15849
- C13, C15: JLCPCB C12530 -> (none); LCSC (none) -> C12530
- C14: JLCPCB C15195 -> (none); LCSC (none) -> C15195
- C16: JLCPCB C14663 -> (none); LCSC (none) -> C14663
- C2, C3: JLCPCB C1547 -> (none); LCSC (none) -> C1547
- C4: JLCPCB C19702 -> (none); LCSC (none) -> C19702
- C6: JLCPCB C13585 -> (none); LCSC (none) -> C13585
- C7: JLCPCB C1848 -> (none); LCSC (none) -> C1848
- D1: JLCPCB C784540 -> (none); LCSC (none) -> C784540
- J2: JLCPCB C324724 -> (none); LCSC (none) -> C324724
- J4: JLCPCB C165948 -> (none); LCSC (none) -> C165948
- L1: JLCPCB C408412 -> (none); LCSC (none) -> C408412
- L2: JLCPCB C26443 -> (none); LCSC (none) -> C26443
- LS1: JLCPCB C391035 -> (none); LCSC (none) -> C391035
- Q1, Q2: JLCPCB C347484 -> (none); LCSC (none) -> C347484
- Q3: JLCPCB C8492 -> (none); LCSC (none) -> C8492
- R10: JLCPCB C11702 -> (none); LCSC (none) -> C11702
- R11, R12, R13: JLCPCB C25104 -> (none); LCSC (none) -> C25104
- R14, R15, R16: JLCPCB C25767 -> (none); LCSC (none) -> C25767
- R17, R18: JLCPCB C25905 -> (none); LCSC (none) -> C25905
- R19, R7: JLCPCB C21189 -> (none); LCSC (none) -> C21189
- R2, R8: JLCPCB C25744 -> (none); LCSC (none) -> C25744
- R20, R21, R23, R24: JLCPCB C25765 -> (none); LCSC (none) -> C25765
- R22: JLCPCB C25741 -> (none); LCSC (none) -> C25741
- R3: JLCPCB C21190 -> (none); LCSC (none) -> C21190
- R4, R5: JLCPCB C23138 -> (none); LCSC (none) -> C23138
- R6: JLCPCB C22975 -> (none); LCSC (none) -> C22975
- R9: JLCPCB C25076 -> (none); LCSC (none) -> C25076
- SW1, SW2, SW3: JLCPCB C221880 -> (none); LCSC (none) -> C221880
- U1: JLCPCB C9051 -> (none); LCSC (none) -> C9051
- U2: JLCPCB C462648 -> (none); LCSC (none) -> C462648
- U3: JLCPCB C465977 -> (none); LCSC (none) -> C465977
- U4: JLCPCB C2827654 -> (none); LCSC (none) -> C2827654
- Y1: JLCPCB C32346 -> (none); LCSC (none) -> C32346
